Commit message: Automatic update of urdf triggered by GitHub Action
r1-models = 4efb1bfe25fcfe6defa0a5eabdc8692ae36c123c
cad-libraries    = https://github.com/icub-tech-iit/cad-libraries/commit/f5522204eb73c981c8722c15328c65abaf0c1f7f
cad-mechanics    = https://github.com/icub-tech-iit/cad-mechanics/commit/7221fbdf8a6d1332bf47bfb82cc037e8c1ac252e
creo2urdf        = https://github.com/icub-tech-iit/creo2urdf/releases/tag/v0.5.11

File: urdf/R1Mk3/robots/R1Mk3Gazebo_minContacts/model.urdf (robot description, URDF)
Before this commit: robot R1Mk3, 182 links, 181 joints
Links:
- link chest_link: geometry collision mesh filename=package://R1Mk3/meshes/simmechanics/sim_emorph_chest.stl scale=0.001 0.001 0.001; visual mesh filename=package://R1Mk3/meshes/simmechanics/sim_emorph_chest.stl scale=0.001 0.001 0.001
- link head_link: geometry collision mesh filename=package://R1Mk3/meshes/simmechanics/sim_cer_emorph_head.stl scale=0.001 0.001 0.001; visual mesh filename=package://R1Mk3/meshes/simmechanics/sim_cer_emorph_head.stl scale=0.001 0.001 0.001
- link l_forearm: geometry collision mesh filename=package://R1Mk3/meshes/simmechanics/sim_emorph_l_forearm.stl scale=0.001 0.001 0.001; visual mesh filename=package://R1Mk3/meshes/simmechanics/sim_emorph_l_forearm.stl scale=0.001 0.001 0.001
- link l_hand_index_1: geometry collision mesh filename=package://R1Mk3/meshes/simmechanics/sim_emorph_l_hand_index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 scale=0.001 0.001 0.001; visual mesh filename=package://R1Mk3/meshes/simmechanics/sim_emorph_l_hand_index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 scale=0.001 0.001 0.001
- link l_hand_index_2: geometry collision mesh filename=package://R1Mk3/meshes/simmechanics/sim_emorph_l_hand_index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 scale=0.001 0.001 0.001; visual mesh filename=package://R1Mk3/meshes/simmechanics/sim_emorph_l_hand_index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 scale=0.001 0.001 0.001
- link l_hand_index_3: geometry collision mesh filename=package://R1Mk3/meshes/simmechanics/sim_emorph_l_hand_index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 scale=0.001 0.001 0.001; visual mesh filename=package://R1Mk3/meshes/simmechanics/sim_emorph_l_hand_index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 scale=0.001 0.001 0.001
- link l_hand_middle_1: geometry collision mesh filename=package://R1Mk3/meshes/simmechanics/sim_emorph_l_hand_middl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 scale=0.001 0.001 0.001; visual mesh filename=package://R1Mk3/meshes/simmechanics/sim_emorph_l_hand_middl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 scale=0.001 0.001 0.001
- link l_hand_middle_2: geometry collision mesh filename=package://R1Mk3/meshes/simmechanics/sim_emorph_l_hand_middl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 scale=0.001 0.001 0.001; visual mesh filename=package://R1Mk3/meshes/simmechanics/sim_emorph_l_hand_middl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 scale=0.001 0.001 0.001
- link l_hand_palm: geometry collision mesh filename=package://R1Mk3/meshes/simmechanics/sim_emorph_l_hand_palm.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 scale=0.001 0.001 0.001; visual mesh filename=package://R1Mk3/meshes/simmechanics/sim_emorph_l_hand_palm.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 scale=0.001 0.001 0.001
- link l_hand_pinkie_1: geometry collision mesh filename=package://R1Mk3/meshes/simmechanics/sim_emorph_l_hand_pinki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 scale=0.001 0.001 0.001; visual mesh filename=package://R1Mk3/meshes/simmechanics/sim_emorph_l_hand_pinki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 scale=0.001 0.001 0.001
- link l_hand_pinkie_2: geometry collision mesh filename=package://R1Mk3/meshes/simmechanics/sim_emorph_l_hand_pinki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 scale=0.001 0.001 0.001; visual mesh filename=package://R1Mk3/meshes/simmechanics/sim_emorph_l_hand_pinki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 scale=0.001 0.001 0.001
- link l_hand_ring_1: geometry collision mesh filename=package://R1Mk3/meshes/simmechanics/sim_emorph_l_hand_ring_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 scale=0.001 0.001 0.001; visual mesh filename=package://R1Mk3/meshes/simmechanics/sim_emorph_l_hand_ring_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 scale=0.001 0.001 0.001
- link l_hand_ring_2: geometry collision mesh filename=package://R1Mk3/meshes/simmechanics/sim_emorph_l_hand_ring_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 scale=0.001 0.001 0.001; visual mesh filename=package://R1Mk3/meshes/simmechanics/sim_emorph_l_hand_ring_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 scale=0.001 0.001 0.001
- link l_hand_thumb_1: geometry collision mesh filename=package://R1Mk3/meshes/simmechanics/sim_emorph_l_hand_thumb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 scale=0.001 0.001 0.001; visual mesh filename=package://R1Mk3/meshes/simmechanics/sim_emorph_l_hand_thumb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 scale=0.001 0.001 0.001
- link l_hand_thumb_2: geometry collision mesh filename=package://R1Mk3/meshes/simmechanics/sim_emorph_l_hand_thumb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 scale=0.001 0.001 0.001; visual mesh filename=package://R1Mk3/meshes/simmechanics/sim_emorph_l_hand_thumb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 scale=0.001 0.001 0.001
- link l_hand_thumb_3: geometry collision mesh filename=package://R1Mk3/meshes/simmechanics/sim_emorph_l_hand_thumb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 scale=0.001 0.001 0.001; visual mesh filename=package://R1Mk3/meshes/simmechanics/sim_emorph_l_hand_thumb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 scale=0.001 0.001 0.001
- link l_shoulder_1: geometry collision mesh filename=package://R1Mk3/meshes/simmechanics/sim_emorph_l_shoulder_1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 scale=0.001 0.001 0.001; visual mesh filename=package://R1Mk3/meshes/simmechanics/sim_emorph_l_shoulder_1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 scale=0.001 0.001 0.001
- link l_shoulder_2: geometry collision mesh filename=package://R1Mk3/meshes/simmechanics/sim_emorph_l_shoulder_2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 scale=0.001 0.001 0.001; visual mesh filename=package://R1Mk3/meshes/simmechanics/sim_emorph_l_shoulder_2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 scale=0.001 0.001 0.001
- link l_shoulder_3: geometry collision mesh filename=package://R1Mk3/meshes/simmechanics/sim_emorph_l_shoulder_3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 scale=0.001 0.001 0.001; visual mesh filename=package://R1Mk3/meshes/simmechanics/sim_emorph_l_shoulder_3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 scale=0.001 0.001 0.001
- link l_upper_arm: geometry collision mesh filename=package://R1Mk3/meshes/simmechanics/sim_emorph_l_upperarm.s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 scale=0.001 0.001 0.001; visual mesh filename=package://R1Mk3/meshes/simmechanics/sim_emorph_l_upperarm.s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 scale=0.001 0.001 0.001
- link l_wrist_1: geometry collision mesh filename=package://R1Mk3/meshes/simmechanics/sim_emorph_l_wrist_1.stl scale=0.001 0.001 0.001; visual mesh filename=package://R1Mk3/meshes/simmechanics/sim_emorph_l_wrist_1.stl scale=0.001 0.001 0.001
- link l_wrist_2: geometry collision mesh filename=package://R1Mk3/meshes/simmechanics/sim_emorph_l_wrist_2.stl scale=0.001 0.001 0.001; visual mesh filename=package://R1Mk3/meshes/simmechanics/sim_emorph_l_wrist_2.stl scale=0.001 0.001 0.001
- link mobile_base_body_link: geometry collision mesh filename=package://R1Mk3/meshes/simmechanics/sim_emorph_mob_base_bod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 scale=0.001 0.001 0.001; visual mesh filename=package://R1Mk3/meshes/simmechanics/sim_emorph_mob_base_bod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 scale=0.001 0.001 0.001
- link neck_link: geometry collision mesh filename=package://R1Mk3/meshes/simmechanics/sim_cer_emorph_neck.stl scale=0.001 0.001 0.001; visual mesh filename=package://R1Mk3/meshes/simmechanics/sim_cer_emorph_neck.stl scale=0.001 0.001 0.001
- link r_forearm: geometry collision mesh filename=package://R1Mk3/meshes/simmechanics/sim_emorph_r_forearm.stl scale=0.001 0.001 0.001; visual mesh filename=package://R1Mk3/meshes/simmechanics/sim_emorph_r_forearm.stl scale=0.001 0.001 0.001
- link r_hand_index_1: geometry collision mesh filename=package://R1Mk3/meshes/simmechanics/sim_emorph_r_hand_index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 scale=0.001 0.001 0.001; visual mesh filename=package://R1Mk3/meshes/simmechanics/sim_emorph_r_hand_index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 scale=0.001 0.001 0.001
- link r_hand_index_2: geometry collision mesh filename=package://R1Mk3/meshes/simmechanics/sim_emorph_r_hand_index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 scale=0.001 0.001 0.001; visual mesh filename=package://R1Mk3/meshes/simmechanics/sim_emorph_r_hand_index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 scale=0.001 0.001 0.001
- link r_hand_index_3: geometry collision mesh filename=package://R1Mk3/meshes/simmechanics/sim_emorph_r_hand_index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 scale=0.001 0.001 0.001; visual mesh filename=package://R1Mk3/meshes/simmechanics/sim_emorph_r_hand_index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 scale=0.001 0.001 0.001
- link r_hand_middle_1: geometry collision mesh filename=package://R1Mk3/meshes/simmechanics/sim_emorph_r_hand_middl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 scale=0.001 0.001 0.001; visual mesh filename=package://R1Mk3/meshes/simmechanics/sim_emorph_r_hand_middl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 scale=0.001 0.001 0.001
- link r_hand_middle_2: geometry collision mesh filename=package://R1Mk3/meshes/simmechanics/sim_emorph_r_hand_middl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 scale=0.001 0.001 0.001; visual mesh filename=package://R1Mk3/meshes/simmechanics/sim_emorph_r_hand_middl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 scale=0.001 0.001 0.001
- link r_hand_palm: geometry collision mesh filename=package://R1Mk3/meshes/simmechanics/sim_emorph_r_hand_palm.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 scale=0.001 0.001 0.001; visual mesh filename=package://R1Mk3/meshes/simmechanics/sim_emorph_r_hand_palm.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 scale=0.001 0.001 0.001
- link r_hand_pinkie_1: geometry collision mesh filename=package://R1Mk3/meshes/simmechanics/sim_emorph_r_hand_pinki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 scale=0.001 0.001 0.001; visual mesh filename=package://R1Mk3/meshes/simmechanics/sim_emorph_r_hand_pinki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 scale=0.001 0.001 0.001
- link r_hand_pinkie_2: geometry collision mesh filename=package://R1Mk3/meshes/simmechanics/sim_emorph_r_hand_pinki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 scale=0.001 0.001 0.001; visual mesh filename=package://R1Mk3/meshes/simmechanics/sim_emorph_r_hand_pinki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 scale=0.001 0.001 0.001
- link r_hand_ring_1: geometry collision mesh filename=package://R1Mk3/meshes/simmechanics/sim_emorph_r_hand_ring_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 scale=0.001 0.001 0.001; visual mesh filename=package://R1Mk3/meshes/simmechanics/sim_emorph_r_hand_ring_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 scale=0.001 0.001 0.001
- link r_hand_ring_2: geometry collision mesh filename=package://R1Mk3/meshes/simmechanics/sim_emorph_r_hand_ring_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 scale=0.001 0.001 0.001; visual mesh filename=package://R1Mk3/meshes/simmechanics/sim_emorph_r_hand_ring_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 scale=0.001 0.001 0.001
- link r_hand_thumb_1: geometry collision mesh filename=package://R1Mk3/meshes/simmechanics/sim_emorph_r_hand_thumb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 scale=0.001 0.001 0.001; visual mesh filename=package://R1Mk3/meshes/simmechanics/sim_emorph_r_hand_thumb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 scale=0.001 0.001 0.001
- link r_hand_thumb_2: geometry collision mesh filename=package://R1Mk3/meshes/simmechanics/sim_emorph_r_hand_thumb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 scale=0.001 0.001 0.001; visual mesh filename=package://R1Mk3/meshes/simmechanics/sim_emorph_r_hand_thumb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 scale=0.001 0.001 0.001
- link r_hand_thumb_3: geometry collision mesh filename=package://R1Mk3/meshes/simmechanics/sim_emorph_r_hand_thumb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 scale=0.001 0.001 0.001; visual mesh filename=package://R1Mk3/meshes/simmechanics/sim_emorph_r_hand_thumb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 scale=0.001 0.001 0.001
- link r_shoulder_1: geometry collision mesh filename=package://R1Mk3/meshes/simmechanics/sim_emorph_r_shoulder_1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 scale=0.001 0.001 0.001; visual mesh filename=package://R1Mk3/meshes/simmechanics/sim_emorph_r_shoulder_1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 scale=0.001 0.001 0.001
- link r_shoulder_2: geometry collision mesh filename=package://R1Mk3/meshes/simmechanics/sim_emorph_r_shoulder_2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 scale=0.001 0.001 0.001; visual mesh filename=package://R1Mk3/meshes/simmechanics/sim_emorph_r_shoulder_2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 scale=0.001 0.001 0.001
- link r_shoulder_3: geometry collision mesh filename=package://R1Mk3/meshes/simmechanics/sim_emorph_r_shoulder_3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 scale=0.001 0.001 0.001; visual mesh filename=package://R1Mk3/meshes/simmechanics/sim_emorph_r_shoulder_3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 scale=0.001 0.001 0.001
- link r_upper_arm: geometry collision mesh filename=package://R1Mk3/meshes/simmechanics/sim_emorph_r_upperarm.s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 scale=0.001 0.001 0.001; visual mesh filename=package://R1Mk3/meshes/simmechanics/sim_emorph_r_upperarm.s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 scale=0.001 0.001 0.001
- link r_wrist_1: geometry collision mesh filename=package://R1Mk3/meshes/simmechanics/sim_emorph_r_wrist_1.stl scale=0.001 0.001 0.001; visual mesh filename=package://R1Mk3/meshes/simmechanics/sim_emorph_r_wrist_1.stl scale=0.001 0.001 0.001
- link r_wrist_2: geometry collision mesh filename=package://R1Mk3/meshes/simmechanics/sim_emorph_r_wrist_2.stl scale=0.001 0.001 0.001; visual mesh filename=package://R1Mk3/meshes/simmechanics/sim_emorph_r_wrist_2.stl scale=0.001 0.001 0.001
- link torso_pin_eq_link: geometry collision mesh filename=package://R1Mk3/meshes/simmechanics/sim_emorph_torso_pin_eq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 scale=0.001 0.001 0.001; visual mesh filename=package://R1Mk3/meshes/simmechanics/sim_emorph_torso_pin_eq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 scale=0.001 0.001 0.001
- link torso_platform_link: geometry collision mesh filename=package://R1Mk3/meshes/simmechanics/sim_emorph_torso_platfo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 scale=0.001 0.001 0.001; visual mesh filename=package://R1Mk3/meshes/simmechanics/sim_emorph_torso_platfo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 scale=0.001 0.001 0.001
- link torso_slider_eq_link: geometry collision mesh filename=package://R1Mk3/meshes/simmechanics/sim_emorph_torso_slider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 scale=0.001 0.001 0.001; visual mesh filename=package://R1Mk3/meshes/simmechanics/sim_emorph_torso_slider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 scale=0.001 0.001 0.001

Commit message: Automatic update of urdf triggered by GitHub Action
r1-models = 4efb1bfe25fcfe6defa0a5eabdc8692ae36c123c
cad-libraries    = https://github.com/icub-tech-iit/cad-libraries/commit/f5522204eb73c981c8722c15328c65abaf0c1f7f
cad-mechanics    = https://github.com/icub-tech-iit/cad-mechanics/commit/7221fbdf8a6d1332bf47bfb82cc037e8c1ac252e
creo2urdf        = https://github.com/icub-tech-iit/creo2urdf/releases/tag/v0.5.11

File: urdf/R1Mk3/robots/R1Mk3Gazebo_minContacts/model.urdf (robot description, URDF)
Before this commit: robot R1Mk3, 182 links, 181 joints
Links:
- link chest_link: geometry visual mesh filename=package://R1Mk3/meshes/simmechanics/sim_emorph_chest.stl scale=0.001 0.001 0.001
- link head_link: geometry visual mesh filename=package://R1Mk3/meshes/simmechanics/sim_cer_emorph_head.stl scale=0.001 0.001 0.001
- link l_forearm: geometry visual mesh filename=package://R1Mk3/meshes/simmechanics/sim_emorph_l_forearm.stl scale=0.001 0.001 0.001
- link l_hand_index_1: geometry visual mesh filename=package://R1Mk3/meshes/simmechanics/sim_emorph_l_hand_index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 scale=0.001 0.001 0.001
- link l_hand_index_2: geometry visual mesh filename=package://R1Mk3/meshes/simmechanics/sim_emorph_l_hand_index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 scale=0.001 0.001 0.001
- link l_hand_index_3: geometry visual mesh filename=package://R1Mk3/meshes/simmechanics/sim_emorph_l_hand_index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 scale=0.001 0.001 0.001
- link l_hand_middle_1: geometry visual mesh filename=package://R1Mk3/meshes/simmechanics/sim_emorph_l_hand_middl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 scale=0.001 0.001 0.001
- link l_hand_middle_2: geometry visual mesh filename=package://R1Mk3/meshes/simmechanics/sim_emorph_l_hand_middl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 scale=0.001 0.001 0.001
- link l_hand_palm: geometry visual mesh filename=package://R1Mk3/meshes/simmechanics/sim_emorph_l_hand_palm.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 scale=0.001 0.001 0.001
- link l_hand_pinkie_1: geometry visual mesh filename=package://R1Mk3/meshes/simmechanics/sim_emorph_l_hand_pinki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 scale=0.001 0.001 0.001
- link l_hand_pinkie_2: geometry visual mesh filename=package://R1Mk3/meshes/simmechanics/sim_emorph_l_hand_pinki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 scale=0.001 0.001 0.001
- link l_hand_ring_1: geometry visual mesh filename=package://R1Mk3/meshes/simmechanics/sim_emorph_l_hand_ring_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 scale=0.001 0.001 0.001
- link l_hand_ring_2: geometry visual mesh filename=package://R1Mk3/meshes/simmechanics/sim_emorph_l_hand_ring_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 scale=0.001 0.001 0.001
- link l_hand_thumb_1: geometry visual mesh filename=package://R1Mk3/meshes/simmechanics/sim_emorph_l_hand_thumb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 scale=0.001 0.001 0.001
- link l_hand_thumb_2: geometry visual mesh filename=package://R1Mk3/meshes/simmechanics/sim_emorph_l_hand_thumb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 scale=0.001 0.001 0.001
- link l_hand_thumb_3: geometry visual mesh filename=package://R1Mk3/meshes/simmechanics/sim_emorph_l_hand_thumb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 scale=0.001 0.001 0.001
- link l_shoulder_1: geometry visual mesh filename=package://R1Mk3/meshes/simmechanics/sim_emorph_l_shoulder_1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 scale=0.001 0.001 0.001
- link l_shoulder_2: geometry visual mesh filename=package://R1Mk3/meshes/simmechanics/sim_emorph_l_shoulder_2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 scale=0.001 0.001 0.001
- link l_shoulder_3: geometry visual mesh filename=package://R1Mk3/meshes/simmechanics/sim_emorph_l_shoulder_3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 scale=0.001 0.001 0.001
- link l_upper_arm: geometry visual mesh filename=package://R1Mk3/meshes/simmechanics/sim_emorph_l_upperarm.s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 scale=0.001 0.001 0.001
- link l_wrist_1: geometry visual mesh filename=package://R1Mk3/meshes/simmechanics/sim_emorph_l_wrist_1.stl scale=0.001 0.001 0.001
- link l_wrist_2: geometry visual mesh filename=package://R1Mk3/meshes/simmechanics/sim_emorph_l_wrist_2.stl scale=0.001 0.001 0.001
- link mobile_base_body_link: geometry visual mesh filename=package://R1Mk3/meshes/simmechanics/sim_emorph_mob_base_bod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 scale=0.001 0.001 0.001
- link neck_link: geometry visual mesh filename=package://R1Mk3/meshes/simmechanics/sim_cer_emorph_neck.stl scale=0.001 0.001 0.001
- link r_forearm: geometry visual mesh filename=package://R1Mk3/meshes/simmechanics/sim_emorph_r_forearm.stl scale=0.001 0.001 0.001
- link r_hand_index_1: geometry visual mesh filename=package://R1Mk3/meshes/simmechanics/sim_emorph_r_hand_index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 scale=0.001 0.001 0.001
- link r_hand_index_2: geometry visual mesh filename=package://R1Mk3/meshes/simmechanics/sim_emorph_r_hand_index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 scale=0.001 0.001 0.001
- link r_hand_index_3: geometry visual mesh filename=package://R1Mk3/meshes/simmechanics/sim_emorph_r_hand_index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 scale=0.001 0.001 0.001
- link r_hand_middle_1: geometry visual mesh filename=package://R1Mk3/meshes/simmechanics/sim_emorph_r_hand_middl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 scale=0.001 0.001 0.001
- link r_hand_middle_2: geometry visual mesh filename=package://R1Mk3/meshes/simmechanics/sim_emorph_r_hand_middl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 scale=0.001 0.001 0.001
- link r_hand_palm: geometry visual mesh filename=package://R1Mk3/meshes/simmechanics/sim_emorph_r_hand_palm.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 scale=0.001 0.001 0.001
- link r_hand_pinkie_1: geometry visual mesh filename=package://R1Mk3/meshes/simmechanics/sim_emorph_r_hand_pinki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 scale=0.001 0.001 0.001
- link r_hand_pinkie_2: geometry visual mesh filename=package://R1Mk3/meshes/simmechanics/sim_emorph_r_hand_pinki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 scale=0.001 0.001 0.001
- link r_hand_ring_1: geometry visual mesh filename=package://R1Mk3/meshes/simmechanics/sim_emorph_r_hand_ring_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 scale=0.001 0.001 0.001
- link r_hand_ring_2: geometry visual mesh filename=package://R1Mk3/meshes/simmechanics/sim_emorph_r_hand_ring_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 scale=0.001 0.001 0.001
- link r_hand_thumb_1: geometry visual mesh filename=package://R1Mk3/meshes/simmechanics/sim_emorph_r_hand_thumb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 scale=0.001 0.001 0.001
- link r_hand_thumb_2: geometry visual mesh filename=package://R1Mk3/meshes/simmechanics/sim_emorph_r_hand_thumb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 scale=0.001 0.001 0.001
- link r_hand_thumb_3: geometry visual mesh filename=package://R1Mk3/meshes/simmechanics/sim_emorph_r_hand_thumb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 scale=0.001 0.001 0.001
- link r_shoulder_1: geometry visual mesh filename=package://R1Mk3/meshes/simmechanics/sim_emorph_r_shoulder_1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 scale=0.001 0.001 0.001
- link r_shoulder_2: geometry visual mesh filename=package://R1Mk3/meshes/simmechanics/sim_emorph_r_shoulder_2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 scale=0.001 0.001 0.001
- link r_shoulder_3: geometry visual mesh filename=package://R1Mk3/meshes/simmechanics/sim_emorph_r_shoulder_3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 scale=0.001 0.001 0.001
- link r_upper_arm: geometry visual mesh filename=package://R1Mk3/meshes/simmechanics/sim_emorph_r_upperarm.s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 scale=0.001 0.001 0.001
- link r_wrist_1: geometry visual mesh filename=package://R1Mk3/meshes/simmechanics/sim_emorph_r_wrist_1.stl scale=0.001 0.001 0.001
- link r_wrist_2: geometry visual mesh filename=package://R1Mk3/meshes/simmechanics/sim_emorph_r_wrist_2.stl scale=0.001 0.001 0.001
- link torso_pin_eq_link: geometry visual mesh filename=package://R1Mk3/meshes/simmechanics/sim_emorph_torso_pin_eq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 scale=0.001 0.001 0.001
- link torso_platform_link: geometry visual mesh filename=package://R1Mk3/meshes/simmechanics/sim_emorph_torso_platfo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 scale=0.001 0.001 0.001
- link torso_slider_eq_link: geometry visual mesh filename=package://R1Mk3/meshes/simmechanics/sim_emorph_torso_slider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 scale=0.001 0.001 0.001

Commit message: Fix minContacts model
It fixes #14

File: urdf/R1Mk3/robots/R1Mk3Gazebo_minContacts/model.urdf (robot description, URDF)
Before this commit: robot R1Mk3, 182 links, 181 joints
Links:
- link mobile_base_body_link: geometry collision mesh filename=package://R1Mk3/meshes/simmechanics/sim_emorph_mob_base_bod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 scale=0.001 0.001 0.001; visual mesh filename=package://R1Mk3/meshes/simmechanics/sim_emorph_mob_base_bod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 scale=0.001 0.001 0.001
