Commit message: Add r1-model-test

File: urdf/R1Mk3/robots/R1Mk3Gazebo/model.urdf (robot description, URDF)
Before this commit: robot R1Mk3, 180 links, 179 joints
Links:
- added link l_arm_ft
- added link r_arm_ft
Joints:
- added joint l_arm_ft_fixed_joint: type fixed, parent l_shoulder_2, child l_arm_ft, origin xyz=-0.0043499999999990074 0.015000000000000069 -0.08430000000000004 rpy=3.14159265358978 -8.827137882952753e-17 -1.5707963267948901
- added joint r_arm_ft_fixed_joint: type fixed, parent r_shoulder_2, child r_arm_ft, origin xyz=-0.0068499999999994746 -0.015000000000000041 -0.08429999999999993 rpy=-3.1415926535897865 1.4451318944920141e-16 1.5707963267948946

Commit message: Automatic update of urdf triggered by GitHub Action
r1-models = 145a45800e94897517a9957871af82b6e54bc47a
cad-libraries    = https://github.com/icub-tech-iit/cad-libraries/commit/c8d497f76c0115af3bd53f7a28ff41e273e46800
cad-mechanics    = https://github.com/icub-tech-iit/cad-mechanics/commit/02a8f13785a3ef1320a4d4f97012ae967b847b9b
creo2urdf        = https://github.com/icub-tech-iit/creo2urdf/releases/tag/v0.5.6

File: urdf/R1Mk3/robots/R1Mk3Gazebo/model.urdf (robot description, URDF)
Before this commit: robot R1Mk3, 182 links, 181 joints
Joints:
- joint l_elbow: limit lower=-0.05235987755982989 upper=1.3089969389957472 effort=1e+9 velocity=1e+9 -> lower=-0.08726646259971647 upper=2.0943951023931953 effort=1e+9 velocity=1e+9
- joint l_shoulder_yaw: limit lower=-0.8726646259971648 upper=1.3962634015954636 effort=1e+9 velocity=1e+9 -> lower=-0.9075712110370514 upper=1.4311699866353502 effort=1e+9 velocity=1e+9
- joint l_wrist_pitch: limit lower=-0.5585053606381855 upper=0.5585053606381855 effort=1e+9 velocity=1e+9 -> lower=-0.3490658503988659 upper=0.3490658503988659 effort=1e+9 velocity=1e+9
- joint l_wrist_roll: limit lower=-1.0821041362364843 upper=0.9075712110370514 effort=1e+9 velocity=1e+9 -> lower=-0.3490658503988659 upper=0.5235987755982988 effort=1e+9 velocity=1e+9
- joint r_elbow: limit lower=-0.05235987755982989 upper=1.3089969389957472 effort=1e+9 velocity=1e+9 -> lower=-0.08726646259971647 upper=2.0943951023931953 effort=1e+9 velocity=1e+9
- joint r_shoulder_yaw: limit lower=-0.8726646259971648 upper=1.3962634015954636 effort=1e+9 velocity=1e+9 -> lower=-0.9075712110370514 upper=1.4311699866353502 effort=1e+9 velocity=1e+9
- joint r_wrist_pitch: limit lower=-0.5585053606381855 upper=0.5585053606381855 effort=1e+9 velocity=1e+9 -> lower=-0.3490658503988659 upper=0.3490658503988659 effort=1e+9 velocity=1e+9
- joint r_wrist_roll: limit lower=-1.0821041362364843 upper=0.9075712110370514 effort=1e+9 velocity=1e+9 -> lower=-0.3490658503988659 upper=0.5235987755982988 effort=1e+9 velocity=1e+9

File: urdf/R1Mk3/robots/R1Mk3Gazebo_minContacts/model.urdf (robot description, URDF)
Before this commit: robot R1Mk3, 182 links, 181 joints
Joints:
- joint l_elbow: limit lower=-0.05235987755982989 upper=1.3089969389957472 effort=1e+9 velocity=1e+9 -> lower=-0.08726646259971647 upper=2.0943951023931953 effort=1e+9 velocity=1e+9
- joint l_shoulder_yaw: limit lower=-0.8726646259971648 upper=1.3962634015954636 effort=1e+9 velocity=1e+9 -> lower=-0.9075712110370514 upper=1.4311699866353502 effort=1e+9 velocity=1e+9
- joint l_wrist_pitch: limit lower=-0.5585053606381855 upper=0.5585053606381855 effort=1e+9 velocity=1e+9 -> lower=-0.3490658503988659 upper=0.3490658503988659 effort=1e+9 velocity=1e+9
- joint l_wrist_roll: limit lower=-1.0821041362364843 upper=0.9075712110370514 effort=1e+9 velocity=1e+9 -> lower=-0.3490658503988659 upper=0.5235987755982988 effort=1e+9 velocity=1e+9
- joint r_elbow: limit lower=-0.05235987755982989 upper=1.3089969389957472 effort=1e+9 velocity=1e+9 -> lower=-0.08726646259971647 upper=2.0943951023931953 effort=1e+9 velocity=1e+9
- joint r_shoulder_yaw: limit lower=-0.8726646259971648 upper=1.3962634015954636 effort=1e+9 velocity=1e+9 -> lower=-0.9075712110370514 upper=1.4311699866353502 effort=1e+9 velocity=1e+9
- joint r_wrist_pitch: limit lower=-0.5585053606381855 upper=0.5585053606381855 effort=1e+9 velocity=1e+9 -> lower=-0.3490658503988659 upper=0.3490658503988659 effort=1e+9 velocity=1e+9
- joint r_wrist_roll: limit lower=-1.0821041362364843 upper=0.9075712110370514 effort=1e+9 velocity=1e+9 -> lower=-0.3490658503988659 upper=0.5235987755982988 effort=1e+9 velocity=1e+9

File: urdf/R1Mk3/robots/R1SN003/model.urdf (robot description, URDF)
Before this commit: robot R1Mk3, 182 links, 181 joints
Joints:
- joint l_elbow: limit lower=-0.05235987755982989 upper=1.3089969389957472 effort=1e+9 velocity=1e+9 -> lower=-0.08726646259971647 upper=2.0943951023931953 effort=1e+9 velocity=1e+9
- joint l_shoulder_yaw: limit lower=-0.8726646259971648 upper=1.3962634015954636 effort=1e+9 velocity=1e+9 -> lower=-0.9075712110370514 upper=1.4311699866353502 effort=1e+9 velocity=1e+9
- joint l_wrist_pitch: limit lower=-0.5585053606381855 upper=0.5585053606381855 effort=1e+9 velocity=1e+9 -> lower=-0.3490658503988659 upper=0.3490658503988659 effort=1e+9 velocity=1e+9
- joint l_wrist_roll: limit lower=-1.0821041362364843 upper=0.9075712110370514 effort=1e+9 velocity=1e+9 -> lower=-0.3490658503988659 upper=0.5235987755982988 effort=1e+9 velocity=1e+9
- joint r_elbow: limit lower=-0.05235987755982989 upper=1.3089969389957472 effort=1e+9 velocity=1e+9 -> lower=-0.08726646259971647 upper=2.0943951023931953 effort=1e+9 velocity=1e+9
- joint r_shoulder_yaw: limit lower=-0.8726646259971648 upper=1.3962634015954636 effort=1e+9 velocity=1e+9 -> lower=-0.9075712110370514 upper=1.4311699866353502 effort=1e+9 velocity=1e+9
- joint r_wrist_pitch: limit lower=-0.5585053606381855 upper=0.5585053606381855 effort=1e+9 velocity=1e+9 -> lower=-0.3490658503988659 upper=0.3490658503988659 effort=1e+9 velocity=1e+9
- joint r_wrist_roll: limit lower=-1.0821041362364843 upper=0.9075712110370514 effort=1e+9 velocity=1e+9 -> lower=-0.3490658503988659 upper=0.5235987755982988 effort=1e+9 velocity=1e+9

Commit message: Automatic update of urdf triggered by GitHub Action
r1-models = a732d6ac1c027e3171caba69679a141b26ec2086
cad-libraries    = https://github.com/icub-tech-iit/cad-libraries/commit/2e5d9fe9b597bcfddd856b19156f111bdeb8c226
cad-mechanics    = https://github.com/icub-tech-iit/cad-mechanics/commit/02a8f13785a3ef1320a4d4f97012ae967b847b9b
creo2urdf        = https://github.com/icub-tech-iit/creo2urdf/releases/tag/v0.5.8

File: urdf/R1Mk3/robots/R1Mk3Gazebo/model.urdf (robot description, URDF)
Before this commit: robot R1Mk3, 182 links, 181 joints
Links:
- link mobile_base_l_tyre_link: geometry collision cylinder length=0.005 radius=0.16; visual mesh filename=package://R1Mk3/meshes/simmechanics/sim_emorph_mobile_base_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 scale=0.001 0.001 0.001
- link mobile_base_r_tyre_link: geometry collision cylinder length=0.005 radius=0.16; visual mesh filename=package://R1Mk3/meshes/simmechanics/sim_emorph_mobile_base_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 scale=0.001 0.001 0.001

File: urdf/R1Mk3/robots/R1Mk3Gazebo_minContacts/model.urdf (robot description, URDF)
Before this commit: robot R1Mk3, 182 links, 181 joints
Links:
- link mobile_base_l_tyre_link: geometry collision mesh filename=package://R1Mk3/meshes/simmechanics/sim_emorph_mobile_base_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 scale=0.001 0.001 0.001; visual mesh filename=package://R1Mk3/meshes/simmechanics/sim_emorph_mobile_base_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 scale=0.001 0.001 0.001
- link mobile_base_r_tyre_link: geometry collision mesh filename=package://R1Mk3/meshes/simmechanics/sim_emorph_mobile_base_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 scale=0.001 0.001 0.001; visual mesh filename=package://R1Mk3/meshes/simmechanics/sim_emorph_mobile_base_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 scale=0.001 0.001 0.001

File: urdf/R1Mk3/robots/R1SN003/model.urdf (robot description, URDF)
Before this commit: robot R1Mk3, 182 links, 181 joints
Links:
- link mobile_base_l_tyre_link: geometry collision cylinder length=0.005 radius=0.16; visual mesh filename=package://R1Mk3/meshes/simmechanics/sim_emorph_mobile_base_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 scale=0.001 0.001 0.001
- link mobile_base_r_tyre_link: geometry collision cylinder length=0.005 radius=0.16; visual mesh filename=package://R1Mk3/meshes/simmechanics/sim_emorph_mobile_base_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 scale=0.001 0.001 0.001

Commit message: Automatic update of urdf triggered by GitHub Action
r1-models = 54ec22f6a88b90b7d1c3e34574299d070a9d0d54
cad-libraries    = https://github.com/icub-tech-iit/cad-libraries/commit/2e5d9fe9b597bcfddd856b19156f111bdeb8c226
cad-mechanics    = https://github.com/icub-tech-iit/cad-mechanics/commit/02a8f13785a3ef1320a4d4f97012ae967b847b9b
creo2urdf        = https://github.com/icub-tech-iit/creo2urdf/releases/tag/v0.5.8

File: urdf/R1Mk3/robots/R1Mk3Gazebo/model.urdf (robot description, URDF)
Before this commit: robot R1Mk3, 182 links, 181 joints
Links:
- link mobile_base_l_tyre_link: geometry collision cylinder length=0.005 radius=0.16; visual mesh filename=package://R1Mk3/meshes/simmechanics/sim_emorph_mobile_base_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 scale=0.001 0.001 0.001
- link mobile_base_r_tyre_link: geometry collision cylinder length=0.005 radius=0.16; visual mesh filename=package://R1Mk3/meshes/simmechanics/sim_emorph_mobile_base_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 scale=0.001 0.001 0.001

File: urdf/R1Mk3/robots/R1SN003/model.urdf (robot description, URDF)
Before this commit: robot R1Mk3, 182 links, 181 joints
Links:
- link mobile_base_l_tyre_link: geometry collision cylinder length=0.005 radius=0.16; visual mesh filename=package://R1Mk3/meshes/simmechanics/sim_emorph_mobile_base_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 scale=0.001 0.001 0.001
- link mobile_base_r_tyre_link: geometry collision cylinder length=0.005 radius=0.16; visual mesh filename=package://R1Mk3/meshes/simmechanics/sim_emorph_mobile_base_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 scale=0.001 0.001 0.001

Commit message: Automatic update of urdf triggered by GitHub Action
r1-models = cd5a9ab873e8ad2ed9beecfb38f98f579372eb74
cad-libraries    = https://github.com/icub-tech-iit/cad-libraries/commit/9a44d055600df8d5472d447dcab1181cc81c51e4
cad-mechanics    = https://github.com/icub-tech-iit/cad-mechanics/commit/02a8f13785a3ef1320a4d4f97012ae967b847b9b
creo2urdf        = https://github.com/icub-tech-iit/creo2urdf/releases/tag/v0.5.9

File: urdf/R1Mk3/robots/R1Mk3Gazebo/model.urdf (robot description, URDF)
Before this commit: robot R1Mk3, 182 links, 181 joints
Links:
- link mobile_base_l_tyre_link: geometry collision cylinder length=0.005 radius=0.16; visual mesh filename=package://R1Mk3/meshes/simmechanics/sim_emorph_mobile_base_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 scale=0.001 0.001 0.001
- link mobile_base_r_tyre_link: geometry collision cylinder length=0.005 radius=0.16; visual mesh filename=package://R1Mk3/meshes/simmechanics/sim_emorph_mobile_base_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 scale=0.001 0.001 0.001
Joints:
- joint mobile_base_l_wheel_joint: limit lower=-6.283185307179586 upper=6.283185307179586 effort=1e+9 velocity=1e+9 -> lower=-1.7453292519943295e+6 upper=1.7453292519943295e+6 effort=1e+9 velocity=1e+9
- joint mobile_base_r_wheel_joint: limit lower=-6.283185307179586 upper=6.283185307179586 effort=1e+9 velocity=1e+9 -> lower=-1.7453292519943295e+6 upper=1.7453292519943295e+6 effort=1e+9 velocity=1e+9

File: urdf/R1Mk3/robots/R1Mk3Gazebo_minContacts/model.urdf (robot description, URDF)
Before this commit: robot R1Mk3, 182 links, 181 joints
Joints:
- joint mobile_base_l_wheel_joint: limit lower=-6.283185307179586 upper=6.283185307179586 effort=1e+9 velocity=1e+9 -> lower=-1.7453292519943295e+6 upper=1.7453292519943295e+6 effort=1e+9 velocity=1e+9
- joint mobile_base_r_wheel_joint: limit lower=-6.283185307179586 upper=6.283185307179586 effort=1e+9 velocity=1e+9 -> lower=-1.7453292519943295e+6 upper=1.7453292519943295e+6 effort=1e+9 velocity=1e+9

File: urdf/R1Mk3/robots/R1SN003/model.urdf (robot description, URDF)
Before this commit: robot R1Mk3, 182 links, 181 joints
Links:
- link mobile_base_l_tyre_link: geometry collision cylinder length=0.005 radius=0.16; visual mesh filename=package://R1Mk3/meshes/simmechanics/sim_emorph_mobile_base_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 scale=0.001 0.001 0.001
- link mobile_base_r_tyre_link: geometry collision cylinder length=0.005 radius=0.16; visual mesh filename=package://R1Mk3/meshes/simmechanics/sim_emorph_mobile_base_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 scale=0.001 0.001 0.001
Joints:
- joint mobile_base_l_wheel_joint: limit lower=-6.283185307179586 upper=6.283185307179586 effort=1e+9 velocity=1e+9 -> lower=-1.7453292519943295e+6 upper=1.7453292519943295e+6 effort=1e+9 velocity=1e+9
- joint mobile_base_r_wheel_joint: limit lower=-6.283185307179586 upper=6.283185307179586 effort=1e+9 velocity=1e+9 -> lower=-1.7453292519943295e+6 upper=1.7453292519943295e+6 effort=1e+9 velocity=1e+9

Commit message: Automatic update of urdf triggered by GitHub Action
r1-models = 723cf925e22963eca38d7e1efe246a170bb34423
cad-libraries    = https://github.com/icub-tech-iit/cad-libraries/commit/9a44d055600df8d5472d447dcab1181cc81c51e4
cad-mechanics    = https://github.com/icub-tech-iit/cad-mechanics/commit/02a8f13785a3ef1320a4d4f97012ae967b847b9b
creo2urdf        = https://github.com/icub-tech-iit/creo2urdf/releases/tag/v0.5.9

File: urdf/R1Mk3/robots/R1Mk3Gazebo/model.urdf (robot description, URDF)
Before this commit: robot R1Mk3, 182 links, 181 joints
Joints:
- joint mobile_base_l_wheel_joint: axis 0 -1 -0 -> 0 1 0
- joint mobile_base_r_wheel_joint: axis -0 -1 -0 -> 0 1 0

File: urdf/R1Mk3/robots/R1Mk3Gazebo_minContacts/model.urdf (robot description, URDF)
Before this commit: robot R1Mk3, 182 links, 181 joints
Joints:
- joint mobile_base_l_wheel_joint: axis 0 -1 -0 -> 0 1 0
- joint mobile_base_r_wheel_joint: axis -0 -1 -0 -> 0 1 0

File: urdf/R1Mk3/robots/R1SN003/model.urdf (robot description, URDF)
Before this commit: robot R1Mk3, 182 links, 181 joints
Joints:
- joint mobile_base_l_wheel_joint: axis 0 -1 -0 -> 0 1 0
- joint mobile_base_r_wheel_joint: axis -0 -1 -0 -> 0 1 0

Commit message: Automatic update of urdf triggered by GitHub Action
r1-models = 38fc876d79711ded862d9da8c5ebad56aa3b155b
cad-libraries    = https://github.com/icub-tech-iit/cad-libraries/commit/a6d3dbe80325b53df059ac2ca4d91137a5addd6b
cad-mechanics    = https://github.com/icub-tech-iit/cad-mechanics/commit/02a8f13785a3ef1320a4d4f97012ae967b847b9b
creo2urdf        = https://github.com/icub-tech-iit/creo2urdf/releases/tag/v0.5.10

File: urdf/R1Mk3/robots/R1Mk3Gazebo/model.urdf (robot description, URDF)
Before this commit: robot R1Mk3, 182 links, 181 joints
Joints:
- joint neck_pitch_joint: axis -1.1561757607518887e-15 -1 5.551115123110952e-17 -> 1.1561757607518887e-15 1 -5.551115123110952e-17
- joint torso_yaw_joint: axis 1.4574786319396409e-16 1.0898835157993226e-15 -1 -> -1.4574786319396409e-16 -1.0898835157993226e-15 1

File: urdf/R1Mk3/robots/R1Mk3Gazebo_minContacts/model.urdf (robot description, URDF)
Before this commit: robot R1Mk3, 182 links, 181 joints
Joints:
- joint neck_pitch_joint: axis -1.1561757607518887e-15 -1 5.551115123110952e-17 -> 1.1561757607518887e-15 1 -5.551115123110952e-17
- joint torso_yaw_joint: axis 1.4574786319396409e-16 1.0898835157993226e-15 -1 -> -1.4574786319396409e-16 -1.0898835157993226e-15 1

File: urdf/R1Mk3/robots/R1SN003/model.urdf (robot description, URDF)
Before this commit: robot R1Mk3, 182 links, 181 joints
Joints:
- joint neck_pitch_joint: axis -1.1561757607518887e-15 -1 5.551115123110952e-17 -> 1.1561757607518887e-15 1 -5.551115123110952e-17
- joint torso_yaw_joint: axis 1.4574786319396409e-16 1.0898835157993226e-15 -1 -> -1.4574786319396409e-16 -1.0898835157993226e-15 1

Commit message: Fixed URDF including double laser

File: urdf/R1Mk3/robots/R1Mk3Gazebo/model.urdf (robot description, URDF)
Before this commit: robot R1Mk3, 182 links, 181 joints
Links:
- removed link mobile_base_lidar
- added link base_laser2_link, mass 0.001
- added link base_laser_link, mass 0.001
- added link mobile_base_double_lidar
- added link mobile_base_lidar_B
- added link mobile_base_lidar_F
- link mobile_base_body_link: geometry collision mesh filename=package://R1Mk3/meshes/obj/sim_cer_mobilebase_body.obj scale=0.001 0.001 0.001; visual mesh filename=package://R1Mk3/meshes/obj/sim_cer_mobilebase_body.obj scale=0.001 0.001 0.001
Joints:
- removed joint mobile_base_lidar_fixed_joint
- added joint base_laser_joint: type fixed, parent mobile_base_body_link, child base_laser_link, origin xyz=0.07 0 0.031 rpy=0 0 0
- added joint base_laser_joint2: type fixed, parent mobile_base_body_link, child base_laser2_link, origin xyz=-0.085 0 0.031 rpy=0 -0 3.14159
- added joint mobile_base_double_lidar_fixed_joint: type fixed, parent mobile_base_body_link, child mobile_base_double_lidar, origin xyz=0.0 0 0.031 rpy=0 0 0
- added joint mobile_base_lidar_B_fixed_joint: type fixed, parent mobile_base_body_link, child mobile_base_lidar_B, origin xyz=-0.085 0 0.031 rpy=0 0 3.14
- added joint mobile_base_lidar_F_fixed_joint: type fixed, parent mobile_base_body_link, child mobile_base_lidar_F, origin xyz=0.07 0 0.031 rpy=0 0 0

Commit message: Automatic update of urdf triggered by GitHub Action
r1-models = cfec47a3b51b8543cbd2d32fe181087914905a6f
cad-libraries    = https://github.com/icub-tech-iit/cad-libraries/commit/5e7c82351458477b3947b0397a72e59532292fe1
cad-mechanics    = https://github.com/icub-tech-iit/cad-mechanics/commit/7221fbdf8a6d1332bf47bfb82cc037e8c1ac252e
creo2urdf        = https://github.com/icub-tech-iit/creo2urdf/releases/tag/v0.5.13

File: urdf/R1Mk3/robots/R1Mk3Gazebo/model.urdf (robot description, URDF)
Before this commit: robot R1Mk3, 182 links, 181 joints
Joints:
- joint base_link_fixed_joint: child mobile_base_body_link -> base_link; parent base_link -> mobile_base_body_link

File: urdf/R1Mk3/robots/R1Mk3Gazebo_minContacts/model.urdf (robot description, URDF)
Before this commit: robot R1Mk3, 182 links, 181 joints
Joints:
- joint base_link_fixed_joint: child mobile_base_body_link -> base_link; parent base_link -> mobile_base_body_link

File: urdf/R1Mk3/robots/R1SN003/model.urdf (robot description, URDF)
Before this commit: robot R1Mk3, 182 links, 181 joints
Joints:
- joint base_link_fixed_joint: child mobile_base_body_link -> base_link; parent base_link -> mobile_base_body_link
