Commit message: Automatic update of urdf triggered by GitHub Action
r1-models = 41b0bcc5209e95ce75e8b9b73486cc9d105999ed
cad-libraries    = https://github.com/icub-tech-iit/cad-libraries/commit/9fe0269d4d782dd6d3b59b77bdcd752e42da0491
cad-mechanics    = https://github.com/icub-tech-iit/cad-mechanics/commit/0cfde9485643d63afeea1019fd3bfdd717589f37
creo2urdf        = https://github.com/icub-tech-iit/creo2urdf/releases/tag/v0.5.14

File: urdf/R1Mk3/robots/R1Mk3Gazebo/model.urdf (robot description, URDF)
Before this commit: robot R1Mk3, 182 links, 181 joints
Links:
- removed link mobile_base_lidar
- added link mobile_base_double_lidar
- added link mobile_base_lidar_B
- added link mobile_base_lidar_F
- link l_hand_thumb_2: mass 0.00669603218404702 -> 0.00744305878263309
- link l_hand_thumb_3: mass 0.006831595 -> 0.00839103052424309
- link mobile_base_body_link: mass 22.387788717205595 -> 22.38733831972927
- link r_hand_thumb_2: mass 0.00669603218404702 -> 0.00744305878263309
- link r_hand_thumb_3: mass 0.00683159462238797 -> 0.008481423658381124
Joints:
- removed joint mobile_base_lidar_fixed_joint
- added joint mobile_base_double_lidar_fixed_joint: type fixed, parent mobile_base_body_link, child mobile_base_double_lidar, origin xyz=0 0 0.031 rpy=0 -0 0
- added joint mobile_base_lidar_B_fixed_joint: type fixed, parent mobile_base_body_link, child mobile_base_lidar_B, origin xyz=-0.085 0 0.031 rpy=0 -0 3.141592653589793
- added joint mobile_base_lidar_F_fixed_joint: type fixed, parent mobile_base_body_link, child mobile_base_lidar_F, origin xyz=0.07 0 0.031 rpy=0 -0 0
- joint l_hand_thumb_skin_0_fixed_joint: origin xyz=0.026405457778888957 -0.002433918058236617 5.551115123125783e-17 rpy=-1.5707963267948963 1.1102230246251565e-16 2.793301925464017 -> xyz=-2.2125551391027898e-11 -0.002433587294553452 -0.026405457778888853 rpy=-1.1609482034540493e-11 -1.2225055986691151 1.5707963268683354
- joint l_hand_thumb_skin_10_fixed_joint: origin xyz=0.032766684597958076 -0.004081940988398508 -0.0032999999999999696 rpy=-1.5707963267948961 -5.551115123125783e-17 -3.075707298047779 -> xyz=-0.003300000023277627 -0.004081610224701271 -0.03276668459736391 rpy=3.1415926535743104 -1.5049109712528579 -1.5707963267955443
- joint l_hand_thumb_skin_11_fixed_joint: origin xyz=0.028280418005286963 -0.0031311476143919825 -0.0032999999999999696 rpy=-1.5707963267948961 -0 2.790891229256258 -> xyz=-0.003300000022465971 -0.0031308168506947176 -0.02828041800469284 rpy=-1.1627790682026587e-11 -1.220094902461357 1.5707963268688572
- joint l_hand_thumb_skin_1_fixed_joint: origin xyz=0.028280418005286963 -0.0031311476143920103 0.0033000000000000806 rpy=-1.5707963267948961 -7.216449660063518e-16 -2.1816615649914324 -> xyz=0.003299999977533996 -0.0031308168507229173 -0.028280418005880898 rpy=3.141592653571252 -0.6108652381980162 -1.570796327023918
- joint l_hand_thumb_skin_2_fixed_joint: origin xyz=0.030192049408458998 -0.0037582416535800467 0 rpy=-1.5707963267948961 -0 2.8764776596464054 -> xyz=-2.2812751687695254e-11 -0.0037579108898968816 -0.030192049408458887 rpy=-1.0975528579504133e-11 -1.305681332851502 1.5707963268508718
- joint l_hand_thumb_skin_3_fixed_joint: origin xyz=0.03276668459795809 -0.004081940988398536 0.003300000000000025 rpy=-1.5707963267948961 -7.216449660063518e-16 -2.1816615649914324 -> xyz=0.0032999999767223676 -0.004081610224729415 -0.03276668459855195 rpy=3.141592653571252 -0.6108652381980161 -1.570796327023918
- joint l_hand_thumb_skin_4_fixed_joint: origin xyz=0.03300000000000006 -0.0011923206886612636 0.005929525942276415 rpy=-3.1415926535897927 3.3306690738754696e-16 -3.1415926535883125 -> xyz=0.005929525918969086 -0.0011919899250033839 -0.03300000000106727 rpy=1.570796323948815 -1.507507555817487 -1.5707963239587988
- joint l_hand_thumb_skin_5_fixed_joint: origin xyz=0.034821366118633415 -0.0034840921633512156 8.326672684688674e-17 rpy=-1.5707963267948963 -2.220446049250313e-16 -2.6595476565932565 -> xyz=-2.364491935580304e-11 -0.0034837613996680783 -0.034821366118633304 rpy=3.141592653576766 -1.0887513297983578 -1.57079632687865
- joint l_hand_thumb_skin_6_fixed_joint: origin xyz=0.036769634404151985 -0.0018288017188734795 0.003300000000000053 rpy=1.5707963267948968 -2.7755575615628914e-16 -2.399827721490722 -> xyz=0.0032999999760114918 -0.0018284709552043588 -0.03676963440474591 rpy=-4.620360040236946e-16 -0.7657426237199224 -1.5707963267949006
- joint l_hand_thumb_skin_7_fixed_joint: origin xyz=0.03825964091188104 -2.9018466437893964e-4 0 rpy=-1.570554204626614 -3.384708831138008e-4 -2.1917443860728234 -> xyz=-2.4250157437677444e-11 -2.898539006957468e-4 -0.038259640911880916 rpy=-3.1415628662062685 -0.620948017682013 -1.5704313693095489
- joint l_hand_thumb_skin_8_fixed_joint: origin xyz=0.03676963440415201 -0.001828801718873424 -0.003299999999999942 rpy=-2.3592109405351698 0.6231239758157896 -2.6159603834403367 -> xyz=-0.0033000000239885308 -0.0018284709551761869 -0.036769634403557905 rpy=3.071469777395219 -0.7763161157147594 -2.432155397543958
- joint l_hand_thumb_skin_9_fixed_joint: origin xyz=0.03300000000000007 -0.0011923206886612636 -0.005929525942276359 rpy=-2.7645689049691455 0.25312544974719003 -3.042753660865159 -> xyz=-0.005929525965583604 -0.0011919899249527854 -0.032999999998932564 rpy=2.9258803345668243 -1.2928372761145006 -2.5531132071417293
- joint l_thumb_add: axis -2.7755575615628914e-16 7.008282842946301e-16 -0.9999999999999999 -> -2.831068712794149e-15 6.453171330633722e-16 -1; origin xyz=0.023374863256390772 -0.0030000000000001414 -0.034523838473554724 rpy=-0.04044970061859073 0.2233191863655339 2.9608435412698353 -> xyz=0.023374863256390335 -0.0029999999999996696 -0.034523838473555835 rpy=-0.040449700618591246 0.22331918636553127 2.960843541269833
- joint l_thumb_dist: axis -2.102484852883521e-15 2.263814136122298e-16 -0.9999999999999993 -> -0.9999999999999997 4.263839635442148e-12 1.8000612565858527e-10; origin xyz=0.03499999999999995 -0.0014999999999998903 -5.551115123125783e-17 rpy=-4.761815941556338e-16 -2.498001805406602e-16 -1.4810340454030065e-12 -> xyz=5.551115123125783e-17 -0.0037106254246526693 -0.034835057900884356 rpy=-0.0632887709773814 1.1102230246251565e-16 2.6684383869213243e-15
- joint l_thumb_prox: axis 5.100087019371813e-16 3.164135620181696e-15 -0.9999999999999997 -> -0.9999999999999998 1.5642875883514762e-11 1.7937541035850657e-10; origin xyz=-0.03809319744959137 -0.0032591938585578573 -0.0036017448035498 rpy=1.3718635850670964 0.1374915277173127 -3.141592653589793 -> xyz=-0.03809319745034652 -0.0032591938585445623 -0.0036017448037202193 rpy=1.430574412172528 -0.1970305979994932 1.5984202269739927
- joint r_hand_thumb_skin_0_fixed_joint: origin xyz=0.02640545777888894 -0.002433918058236617 0 rpy=-1.5707963267948961 2.220446049250313e-16 2.793301925464017 -> xyz=-5.551115123125783e-17 -0.002433587294553591 -0.026405457778889127 rpy=2.765053092553465e-15 -1.22250559866914 1.5707963267948857
- joint r_hand_thumb_skin_10_fixed_joint: origin xyz=0.03276668459795807 -0.00408194098839848 -0.003300000000000025 rpy=-1.5707963267948961 5.551115123125783e-17 -3.075707298047779 -> xyz=-0.003300000000000053 -0.004081610224715565 -0.032766684597958284 rpy=3.141592653589779 -1.5049109712529725 -1.570796326794926
- joint r_hand_thumb_skin_11_fixed_joint: origin xyz=0.028280418005286953 -0.0031311476143919825 -0.0032999999999999974 rpy=-1.5707963267948961 1.6653345369377348e-16 2.790891229256258 -> xyz=-0.003300000000000053 -0.0031308168507090395 -0.02828041800528719 rpy=2.908401871442372e-15 -1.2200949024613812 1.5707963267948855
- joint r_hand_thumb_skin_1_fixed_joint: origin xyz=0.028280418005286932 -0.0031311476143919825 0.003300000000000025 rpy=-1.570796326794896 -7.216449660063518e-16 -2.1816615649914324 -> xyz=0.0032999999999999696 -0.0031308168507089285 -0.02828041800528714 rpy=3.1415926535897922 -0.6108652381980179 -1.5707963267949114
- joint r_hand_thumb_skin_2_fixed_joint: origin xyz=0.030192049408458994 -0.003758241653580019 0 rpy=-1.5707963267948961 2.7755575615628914e-16 2.8764776596464054 -> xyz=0 -0.0037579108898970204 -0.03019204940845916 rpy=3.389732024708853e-15 -1.3056813328515338 1.5707963267948863
- joint r_hand_thumb_skin_3_fixed_joint: origin xyz=0.03276668459795803 -0.004081940988398508 0.0032999999999999974 rpy=-1.570796326794896 -8.326672684688674e-16 -2.1816615649914324 -> xyz=0.0032999999999999974 -0.004081610224715454 -0.032766684597958305 rpy=3.1415926535897922 -0.6108652381980177 -1.5707963267949112
- joint r_hand_thumb_skin_4_fixed_joint: origin xyz=0.03300000000000006 -0.0011923206886612636 0.005929525942276415 rpy=-3.1415926535897927 2.220446049250313e-16 -3.1415926535883125 -> xyz=0.005929525942276387 -0.0011919899249781263 -0.03300000000000026 rpy=1.5707963267948817 -1.507507552842365 -1.5707963267949265
- joint r_hand_thumb_skin_5_fixed_joint: origin xyz=0.03482136611863341 -0.0034840921633512434 0 rpy=-1.5707963267948961 -1.6653345369377348e-16 -2.659547656593256 -> xyz=-5.551115123125783e-17 -0.003483761399668245 -0.034821366118633644 rpy=3.1415926535897913 -1.088751329798369 -1.5707963267949128
- joint r_hand_thumb_skin_6_fixed_joint: origin xyz=0.036769634404151964 -0.0018288017188734518 0.0032999999999999974 rpy=1.570796326794897 -2.220446049250313e-16 -2.399827721490722 -> xyz=0.0032999999999999974 -0.0018284709551903977 -0.036769634404152235 rpy=-1.3861080081060772e-15 -0.7657426207446857 -1.5707963267949117
- joint r_hand_thumb_skin_7_fixed_joint: origin xyz=0.03825964091188099 -2.901846643789119e-4 0 rpy=-1.5705542046266139 -3.3847088311368976e-4 -2.191744386072823 -> xyz=-2.7755575615628914e-17 -2.898539006959133e-4 -0.038259640911881256 rpy=-3.1415628661866624 -0.6209480176820894 -1.570431369087355
- joint r_hand_thumb_skin_8_fixed_joint: origin xyz=0.036769634404152 -0.0018288017188734518 -0.003300000000000025 rpy=-2.3592109405351698 0.6231239758157898 -2.6159603834403367 -> xyz=-0.0032999999999999974 -0.0018284709551905087 -0.03676963440415227 rpy=3.071469774250236 -0.7763161153414891 -2.432155392931655
- joint r_hand_thumb_skin_9_fixed_joint: origin xyz=0.03300000000000001 -0.0011923206886612636 -0.005929525942276359 rpy=-2.7645689049691455 0.25312544974719 -3.042753660865159 -> xyz=-0.005929525942276387 -0.0011919899249783206 -0.03300000000000024 rpy=2.9258803249384773 -1.2928372753400146 -2.553113197096302
- joint r_thumb_add: axis 9.71445146547012e-16 2.542554010709041e-15 0.9999999999999998 -> 4.996003610813204e-16 2.6775506528309486e-15 0.9999999999999999; origin xyz=0.023374863256390613 0.003000000000000197 -0.03452383847355428 rpy=1.7024696942186454e-15 -0.2268928027592651 -6.747454081634266e-16 -> xyz=0.0233748632563905 0.0030000000000003912 -0.03452383847355461 rpy=1.673677624598278e-15 -0.22689280275926468 -4.805912162985855e-17
- joint r_thumb_dist: axis 8.8297424927092e-16 1.174407793238017e-15 -0.9999999999999998 -> -1.0000000000000022 -2.8857703148647843e-14 2.7310966301870412e-16; origin xyz=-0.03499999999999995 0.0014999999999998903 -1.942890293094024e-16 rpy=-3.1398494915180213e-16 -2.7755575615628914e-16 3.141592653588312 -> xyz=-5.551115123125783e-17 -0.003710625528295264 -0.03483505788984388 rpy=-0.0632887739526204 3.164135620181696e-15 1.4696577288475478e-14
- joint r_thumb_prox: axis 1.0928757898653885e-15 -1.0824674490095276e-15 -0.9999999999999997 -> -1.0000000000000009 -1.426636586643326e-14 2.5500435096859064e-15; origin xyz=0.038074654499560476 0.00346910958032548 -0.0036017448035497446 rpy=-1.7697290685226967 -0.1374915277173128 -2.9653796139720434 -> xyz=0.03807465449956053 0.0034691095803252026 -0.0036017448035498 rpy=1.4305744121375041 0.1970305979589347 -1.4222071875351316

File: urdf/R1Mk3/robots/R1Mk3Gazebo_minContacts/model.urdf (robot description, URDF)
Before this commit: robot R1Mk3, 182 links, 181 joints
Links:
- removed link mobile_base_lidar
- added link mobile_base_double_lidar
- added link mobile_base_lidar_B
- added link mobile_base_lidar_F
- link l_hand_thumb_2: mass 0.00669603218404702 -> 0.00744305878263309
- link l_hand_thumb_3: mass 0.006831595 -> 0.00839103052424309
- link mobile_base_body_link: mass 22.387788717205595 -> 22.38733831972927
- link r_hand_thumb_2: mass 0.00669603218404702 -> 0.00744305878263309
- link r_hand_thumb_3: mass 0.00683159462238797 -> 0.008481423658381124
Joints:
- removed joint mobile_base_lidar_fixed_joint
- added joint mobile_base_double_lidar_fixed_joint: type fixed, parent mobile_base_body_link, child mobile_base_double_lidar, origin xyz=0 0 0.031 rpy=0 -0 0
- added joint mobile_base_lidar_B_fixed_joint: type fixed, parent mobile_base_body_link, child mobile_base_lidar_B, origin xyz=-0.085 0 0.031 rpy=0 -0 3.141592653589793
- added joint mobile_base_lidar_F_fixed_joint: type fixed, parent mobile_base_body_link, child mobile_base_lidar_F, origin xyz=0.07 0 0.031 rpy=0 -0 0
- joint l_hand_thumb_skin_0_fixed_joint: origin xyz=0.026405457778888957 -0.002433918058236617 5.551115123125783e-17 rpy=-1.5707963267948963 1.1102230246251565e-16 2.793301925464017 -> xyz=-2.2125551391027898e-11 -0.002433587294553452 -0.026405457778888853 rpy=-1.1609482034540493e-11 -1.2225055986691151 1.5707963268683354
- joint l_hand_thumb_skin_10_fixed_joint: origin xyz=0.032766684597958076 -0.004081940988398508 -0.0032999999999999696 rpy=-1.5707963267948961 -5.551115123125783e-17 -3.075707298047779 -> xyz=-0.003300000023277627 -0.004081610224701271 -0.03276668459736391 rpy=3.1415926535743104 -1.5049109712528579 -1.5707963267955443
- joint l_hand_thumb_skin_11_fixed_joint: origin xyz=0.028280418005286963 -0.0031311476143919825 -0.0032999999999999696 rpy=-1.5707963267948961 -0 2.790891229256258 -> xyz=-0.003300000022465971 -0.0031308168506947176 -0.02828041800469284 rpy=-1.1627790682026587e-11 -1.220094902461357 1.5707963268688572
- joint l_hand_thumb_skin_1_fixed_joint: origin xyz=0.028280418005286963 -0.0031311476143920103 0.0033000000000000806 rpy=-1.5707963267948961 -7.216449660063518e-16 -2.1816615649914324 -> xyz=0.003299999977533996 -0.0031308168507229173 -0.028280418005880898 rpy=3.141592653571252 -0.6108652381980162 -1.570796327023918
- joint l_hand_thumb_skin_2_fixed_joint: origin xyz=0.030192049408458998 -0.0037582416535800467 0 rpy=-1.5707963267948961 -0 2.8764776596464054 -> xyz=-2.2812751687695254e-11 -0.0037579108898968816 -0.030192049408458887 rpy=-1.0975528579504133e-11 -1.305681332851502 1.5707963268508718
- joint l_hand_thumb_skin_3_fixed_joint: origin xyz=0.03276668459795809 -0.004081940988398536 0.003300000000000025 rpy=-1.5707963267948961 -7.216449660063518e-16 -2.1816615649914324 -> xyz=0.0032999999767223676 -0.004081610224729415 -0.03276668459855195 rpy=3.141592653571252 -0.6108652381980161 -1.570796327023918
- joint l_hand_thumb_skin_4_fixed_joint: origin xyz=0.03300000000000006 -0.0011923206886612636 0.005929525942276415 rpy=-3.1415926535897927 3.3306690738754696e-16 -3.1415926535883125 -> xyz=0.005929525918969086 -0.0011919899250033839 -0.03300000000106727 rpy=1.570796323948815 -1.507507555817487 -1.5707963239587988
- joint l_hand_thumb_skin_5_fixed_joint: origin xyz=0.034821366118633415 -0.0034840921633512156 8.326672684688674e-17 rpy=-1.5707963267948963 -2.220446049250313e-16 -2.6595476565932565 -> xyz=-2.364491935580304e-11 -0.0034837613996680783 -0.034821366118633304 rpy=3.141592653576766 -1.0887513297983578 -1.57079632687865
- joint l_hand_thumb_skin_6_fixed_joint: origin xyz=0.036769634404151985 -0.0018288017188734795 0.003300000000000053 rpy=1.5707963267948968 -2.7755575615628914e-16 -2.399827721490722 -> xyz=0.0032999999760114918 -0.0018284709552043588 -0.03676963440474591 rpy=-4.620360040236946e-16 -0.7657426237199224 -1.5707963267949006
- joint l_hand_thumb_skin_7_fixed_joint: origin xyz=0.03825964091188104 -2.9018466437893964e-4 0 rpy=-1.570554204626614 -3.384708831138008e-4 -2.1917443860728234 -> xyz=-2.4250157437677444e-11 -2.898539006957468e-4 -0.038259640911880916 rpy=-3.1415628662062685 -0.620948017682013 -1.5704313693095489
- joint l_hand_thumb_skin_8_fixed_joint: origin xyz=0.03676963440415201 -0.001828801718873424 -0.003299999999999942 rpy=-2.3592109405351698 0.6231239758157896 -2.6159603834403367 -> xyz=-0.0033000000239885308 -0.0018284709551761869 -0.036769634403557905 rpy=3.071469777395219 -0.7763161157147594 -2.432155397543958
- joint l_hand_thumb_skin_9_fixed_joint: origin xyz=0.03300000000000007 -0.0011923206886612636 -0.005929525942276359 rpy=-2.7645689049691455 0.25312544974719003 -3.042753660865159 -> xyz=-0.005929525965583604 -0.0011919899249527854 -0.032999999998932564 rpy=2.9258803345668243 -1.2928372761145006 -2.5531132071417293
- joint l_thumb_add: axis -2.7755575615628914e-16 7.008282842946301e-16 -0.9999999999999999 -> -2.831068712794149e-15 6.453171330633722e-16 -1; origin xyz=0.023374863256390772 -0.0030000000000001414 -0.034523838473554724 rpy=-0.04044970061859073 0.2233191863655339 2.9608435412698353 -> xyz=0.023374863256390335 -0.0029999999999996696 -0.034523838473555835 rpy=-0.040449700618591246 0.22331918636553127 2.960843541269833
- joint l_thumb_dist: axis -2.102484852883521e-15 2.263814136122298e-16 -0.9999999999999993 -> -0.9999999999999997 4.263839635442148e-12 1.8000612565858527e-10; origin xyz=0.03499999999999995 -0.0014999999999998903 -5.551115123125783e-17 rpy=-4.761815941556338e-16 -2.498001805406602e-16 -1.4810340454030065e-12 -> xyz=5.551115123125783e-17 -0.0037106254246526693 -0.034835057900884356 rpy=-0.0632887709773814 1.1102230246251565e-16 2.6684383869213243e-15
- joint l_thumb_prox: axis 5.100087019371813e-16 3.164135620181696e-15 -0.9999999999999997 -> -0.9999999999999998 1.5642875883514762e-11 1.7937541035850657e-10; origin xyz=-0.03809319744959137 -0.0032591938585578573 -0.0036017448035498 rpy=1.3718635850670964 0.1374915277173127 -3.141592653589793 -> xyz=-0.03809319745034652 -0.0032591938585445623 -0.0036017448037202193 rpy=1.430574412172528 -0.1970305979994932 1.5984202269739927
- joint r_hand_thumb_skin_0_fixed_joint: origin xyz=0.02640545777888894 -0.002433918058236617 0 rpy=-1.5707963267948961 2.220446049250313e-16 2.793301925464017 -> xyz=-5.551115123125783e-17 -0.002433587294553591 -0.026405457778889127 rpy=2.765053092553465e-15 -1.22250559866914 1.5707963267948857
- joint r_hand_thumb_skin_10_fixed_joint: origin xyz=0.03276668459795807 -0.00408194098839848 -0.003300000000000025 rpy=-1.5707963267948961 5.551115123125783e-17 -3.075707298047779 -> xyz=-0.003300000000000053 -0.004081610224715565 -0.032766684597958284 rpy=3.141592653589779 -1.5049109712529725 -1.570796326794926
- joint r_hand_thumb_skin_11_fixed_joint: origin xyz=0.028280418005286953 -0.0031311476143919825 -0.0032999999999999974 rpy=-1.5707963267948961 1.6653345369377348e-16 2.790891229256258 -> xyz=-0.003300000000000053 -0.0031308168507090395 -0.02828041800528719 rpy=2.908401871442372e-15 -1.2200949024613812 1.5707963267948855
- joint r_hand_thumb_skin_1_fixed_joint: origin xyz=0.028280418005286932 -0.0031311476143919825 0.003300000000000025 rpy=-1.570796326794896 -7.216449660063518e-16 -2.1816615649914324 -> xyz=0.0032999999999999696 -0.0031308168507089285 -0.02828041800528714 rpy=3.1415926535897922 -0.6108652381980179 -1.5707963267949114
- joint r_hand_thumb_skin_2_fixed_joint: origin xyz=0.030192049408458994 -0.003758241653580019 0 rpy=-1.5707963267948961 2.7755575615628914e-16 2.8764776596464054 -> xyz=0 -0.0037579108898970204 -0.03019204940845916 rpy=3.389732024708853e-15 -1.3056813328515338 1.5707963267948863
- joint r_hand_thumb_skin_3_fixed_joint: origin xyz=0.03276668459795803 -0.004081940988398508 0.0032999999999999974 rpy=-1.570796326794896 -8.326672684688674e-16 -2.1816615649914324 -> xyz=0.0032999999999999974 -0.004081610224715454 -0.032766684597958305 rpy=3.1415926535897922 -0.6108652381980177 -1.5707963267949112
- joint r_hand_thumb_skin_4_fixed_joint: origin xyz=0.03300000000000006 -0.0011923206886612636 0.005929525942276415 rpy=-3.1415926535897927 2.220446049250313e-16 -3.1415926535883125 -> xyz=0.005929525942276387 -0.0011919899249781263 -0.03300000000000026 rpy=1.5707963267948817 -1.507507552842365 -1.5707963267949265
- joint r_hand_thumb_skin_5_fixed_joint: origin xyz=0.03482136611863341 -0.0034840921633512434 0 rpy=-1.5707963267948961 -1.6653345369377348e-16 -2.659547656593256 -> xyz=-5.551115123125783e-17 -0.003483761399668245 -0.034821366118633644 rpy=3.1415926535897913 -1.088751329798369 -1.5707963267949128
- joint r_hand_thumb_skin_6_fixed_joint: origin xyz=0.036769634404151964 -0.0018288017188734518 0.0032999999999999974 rpy=1.570796326794897 -2.220446049250313e-16 -2.399827721490722 -> xyz=0.0032999999999999974 -0.0018284709551903977 -0.036769634404152235 rpy=-1.3861080081060772e-15 -0.7657426207446857 -1.5707963267949117
- joint r_hand_thumb_skin_7_fixed_joint: origin xyz=0.03825964091188099 -2.901846643789119e-4 0 rpy=-1.5705542046266139 -3.3847088311368976e-4 -2.191744386072823 -> xyz=-2.7755575615628914e-17 -2.898539006959133e-4 -0.038259640911881256 rpy=-3.1415628661866624 -0.6209480176820894 -1.570431369087355
- joint r_hand_thumb_skin_8_fixed_joint: origin xyz=0.036769634404152 -0.0018288017188734518 -0.003300000000000025 rpy=-2.3592109405351698 0.6231239758157898 -2.6159603834403367 -> xyz=-0.0032999999999999974 -0.0018284709551905087 -0.03676963440415227 rpy=3.071469774250236 -0.7763161153414891 -2.432155392931655
- joint r_hand_thumb_skin_9_fixed_joint: origin xyz=0.03300000000000001 -0.0011923206886612636 -0.005929525942276359 rpy=-2.7645689049691455 0.25312544974719 -3.042753660865159 -> xyz=-0.005929525942276387 -0.0011919899249783206 -0.03300000000000024 rpy=2.9258803249384773 -1.2928372753400146 -2.553113197096302
- joint r_thumb_add: axis 9.71445146547012e-16 2.542554010709041e-15 0.9999999999999998 -> 4.996003610813204e-16 2.6775506528309486e-15 0.9999999999999999; origin xyz=0.023374863256390613 0.003000000000000197 -0.03452383847355428 rpy=1.7024696942186454e-15 -0.2268928027592651 -6.747454081634266e-16 -> xyz=0.0233748632563905 0.0030000000000003912 -0.03452383847355461 rpy=1.673677624598278e-15 -0.22689280275926468 -4.805912162985855e-17
- joint r_thumb_dist: axis 8.8297424927092e-16 1.174407793238017e-15 -0.9999999999999998 -> -1.0000000000000022 -2.8857703148647843e-14 2.7310966301870412e-16; origin xyz=-0.03499999999999995 0.0014999999999998903 -1.942890293094024e-16 rpy=-3.1398494915180213e-16 -2.7755575615628914e-16 3.141592653588312 -> xyz=-5.551115123125783e-17 -0.003710625528295264 -0.03483505788984388 rpy=-0.0632887739526204 3.164135620181696e-15 1.4696577288475478e-14
- joint r_thumb_prox: axis 1.0928757898653885e-15 -1.0824674490095276e-15 -0.9999999999999997 -> -1.0000000000000009 -1.426636586643326e-14 2.5500435096859064e-15; origin xyz=0.038074654499560476 0.00346910958032548 -0.0036017448035497446 rpy=-1.7697290685226967 -0.1374915277173128 -2.9653796139720434 -> xyz=0.03807465449956053 0.0034691095803252026 -0.0036017448035498 rpy=1.4305744121375041 0.1970305979589347 -1.4222071875351316
